Commit message: updates to arlobot model

File: src/arlobot/arlobot_description/urdf/arlobot.baselevel.urdf.xacro (robot description, xacro)
@@ -4,6 +4,6 @@
     <!--
         The baselevel includes:
-            - Platter with wheel cutout (arlobot.platter.urdf.xacro)
-            - Two casters (front and back)
+            - Platter with wheel cutout (arlobot_description/meshes/arlobot.platterwithcutout.dae)
+            - Two casters (front and back, arlobot_description/meshes/28971-Caster-Wheel-Kit-v1.0.stl)
             - Five forward-facing ultrasonic sensors (arlobot.rangesensor.urdf.xacro)
             - Two forward-facing infrared sensors (arlobot.rangesensor.urdf.xacro)
@@ -16,4 +16,7 @@
     -->
     <!-- The base level macro -->
+    <!-- The base level macro essentially defines the bottom platter of the Arlobot (this is the platter with the cutout
+    for the wheels and forms the base of the robot.  It is the minimum of an Arlobot.
+    -->
     <macro name="baselevel" params="parent name color">
         <joint name="${parent}_${name}_joint" type="fixed">
@@ -38,8 +41,13 @@
         </link>
     </macro>
-    <!-- define the caster -->
+    <!-- The caster macro -->
+    <!-- The caster macro defines provides a definition for the front and back casters.  The mesh for the caster came
+    from Chrisl8's implementation of Arlobot.
+    -->
+    <property name="caster_radius" value="0.18745"/>
     <macro name="caster" params="suffix parent reflect color">
         <joint name="${parent}_${suffix}_caster_joint" type="fixed">
-            <origin xyz="${reflect*0.18745} 0 -0.00475" rpy="0 0 0" />
+            <!-- <origin xyz="${reflect*0.18745} 0 -0.00475" rpy="0 0 0" /> -->
+            <origin xyz="${reflect*caster_radius} 0 ${-platter_height/2}" rpy="0 0 0" />
             <parent link="${parent}_link" />
             <child link="${parent}_${suffix}_caster_link" />
@@ -60,4 +68,8 @@
         </link>
     </macro>
+    <!-- The power distribution macro -->
+    <!-- The power distribution macro defines the power distribution block on the Alrobot.  At present it, it is just
+    a box primitive.
+    -->
     <property name="power_size_x" value="0.08255"/>
     <property name="power_size_y" value="0.1397"/>
@@ -87,4 +99,9 @@
         </link>
     </macro>
+    <!-- The HB25 motor driver macro -->
+    <!-- The HB25 motor driver macro defines the HB-25 motor drivers.  There are two motor drivers and they can be
+    mounted anywhere on Arlobot.  This implementation has them mounted on the back of Arlobot.  At present the
+    display is a box primitive.
+    -->
     <property name="motor_driver_size_x" value="0.03175"/>
     <property name="motor_driver_size_y" value="0.0381"/>
@@ -119,4 +136,9 @@
         </link>
     </macro>
+    <!-- The controller macro -->
+    <!-- The controller macro defines the Arlobot controller components.  Parallax's offering uses a Propeller Acitivity
+    board.  This implementation uses a Raspberry Pi and Two Psoc4M-044 development kits.  The display is a simple box
+    primitive
+    -->
     <property name="controller_size_x" value="0.0635"/>
     <property name="controller_size_y" value="0.1016"/>
@@ -146,4 +168,8 @@
         </link>
     </macro>
+    <!-- The relay macro -->
+    <!-- The relay macro defines a relay bank (8 relays).  Two relays are used to control the HB-25 motor drivers.
+     The display is a simple box primitive
+     -->
     <property name="relay_size_x" value="0.0254"/>
     <property name="relay_size_y" value="0.127"/>
@@ -173,13 +199,18 @@
         </link>
     </macro>
-    <!-- Build the Base Level -->
+    <!--
+    Build the Base Level
+    Below is the build-up of the baselevel component of the Arlobot
+    -->
     <caster parent="baselevel" suffix="front" reflect="1" color="LightGrey"/>
     <caster parent="baselevel" suffix="back" reflect="-1" color="LightGrey"/>
-    <property name="ultrasonic_offset_z" value="${baselevel_top_offset_z + ultrasonic_height/2}"/>
-    <ultrasonic_array_5_front parent="baselevel" offset_z="${ultrasonic_offset_z}"/>
-    <ultrasonic_array_5_back parent="baselevel" offset_z="${ultrasonic_offset_z}"/>
-    <property name="infrared_offset_z" value="${-platter_height - infrared_height/2}"/>
-    <infrared_array_2_front_lower parent="baselevel" offset_z="${infrared_offset_z}"/>
-    <infrared_array_2_back_lower parent="baselevel" offset_z="${infrared_offset_z}"/>
+    <!-- This calculation is needed to position the ultrasonic sensor on the top of the base level platter -->
+    <property name="baselevel_ultrasonic_offset_z" value="${baselevel_top_offset_z + ultrasonic_height/2}"/>
+    <ultrasonic_array_5_front parent="baselevel" offset_z="${baselevel_ultrasonic_offset_z}"/>
+    <ultrasonic_array_5_back parent="baselevel" offset_z="${baselevel_ultrasonic_offset_z}"/>
+    <!-- This calculation is needed to position the infrared sensor under the base level platter -->
+    <property name="baselevel_infrared_offset_z" value="${-platter_height - infrared_height/2}"/>
+    <infrared_array_2_front_lower parent="baselevel" offset_z="${baselevel_infrared_offset_z}"/>
+    <infrared_array_2_back_lower parent="baselevel" offset_z="${baselevel_infrared_offset_z}"/>
     <power parent="baselevel" color="LightGrey"/>
     <motor_driver parent="baselevel" suffix="left" color="Orange" offset_x="${left_motor_driver_offset_x}" offset_y="${left_motor_driver_offset_y}" offset_z="${left_motor_driver_offset_z}"  yaw="${angle_315}"/>

File: src/arlobot/arlobot_description/urdf/arlobot.global.urdf.xacro (robot description, xacro)
@@ -11,33 +11,42 @@
     -->
     <property name="angle_0" value="0"/>
-    <property name="angle_30" value="${PI/6}"/> <!-- 0.5236 -->
-    <property name="angle_45" value="${PI/4}"/> <!-- 0.7854 -->
-    <property name="angle_60" value="${PI/3}"/> <!-- 1.0472 -->
-    <property name="angle_90" value="${PI/2}"/> <!-- 1.0472 -->
-    <property name="angle_120" value="${2*PI/3}"/> <!-- 2.0944 -->
-    <property name="angle_135" value="${3*PI/4}"/> <!-- 2.3562 -->
-    <property name="angle_150" value="${5*PI/6}"/> <!-- 2.6180 -->
-    <property name="angle_180" value="${PI}"/> <!-- 3.1416 -->
-    <property name="angle_210" value="${7*PI/6}"/> <!-- 3.6652 -->
-    <property name="angle_225" value="$(5*PI/4}"/> <!-- 3.9270 -->
-    <property name="angle_240" value="${4*PI/3}"/> <!-- 4.1888 -->
-    <property name="angle_315" value="${7*PI/4}"/> <!-- 5.4978 -->
-    <property name="angle_330" value="${11*PI/6}"/> <!-- 5.7596 -->
-    <property name="angle_300" value="${5*PI/3}"/> <!-- 5.2360 -->
+    <property name="angle_15" value="${PI/12}"/>        <!-- 0.2618 -->
+    <property name="angle_30" value="${PI/6}"/>         <!-- 0.5236 -->
+    <property name="angle_45" value="${PI/4}"/>         <!-- 0.7854 -->
+    <property name="angle_60" value="${PI/3}"/>         <!-- 1.0472 -->
+    <property name="angle_90" value="${PI/2}"/>         <!-- 1.0472 -->
+    <property name="angle_120" value="${2*PI/3}"/>      <!-- 2.0944 -->
+    <property name="angle_135" value="${3*PI/4}"/>      <!-- 2.3562 -->
+    <property name="angle_150" value="${5*PI/6}"/>      <!-- 2.6180 -->
+    <property name="angle_165" value="${11*PI/12}"/>    <!-- 2.8800 -->
+    <property name="angle_180" value="${PI}"/>          <!-- 3.1416 -->
+    <property name="angle_195" value="${13*PI/12}"/>    <!-- 3.4000 -->
+    <property name="angle_210" value="${7*PI/6}"/>      <!-- 3.6652 -->
+    <property name="angle_225" value="${5*PI/4}"/>      <!-- 3.9270 -->
+    <property name="angle_240" value="${4*PI/3}"/>      <!-- 4.1888 -->
+    <property name="angle_300" value="${5*PI/3}"/>      <!-- 5.2360 -->
+    <property name="angle_315" value="${7*PI/4}"/>      <!-- 5.4978 -->
+    <property name="angle_330" value="${11*PI/6}"/>     <!-- 5.7596 -->
+    <property name="angle_345" value="${23*PI/24}"/>    <!-- 5.2360 -->
     <property name="cos_angle_0" value="1.0000"/>
+    <property name="cos_angle_15" value="0.9659"/>
     <property name="cos_angle_30" value="0.8660"/>
     <property name="cos_angle_45" value="0.7071"/>
     <property name="cos_angle_60" value="0.5000"/>
     <property name="cos_angle_120" value="-0.5000"/>
-    <property name="cos_angle_135" value="−0.7071"/>
+    <property name="cos_angle_135" value="-0.7071"/>
     <property name="cos_angle_150" value="-0.8660"/>
+    <property name="cos_angle_165" value="-0.9659"/>
     <property name="cos_angle_180" value="-1.0000"/>
+    <property name="cos_angle_195" value="-0.9659"/>
     <property name="cos_angle_210" value="-0.8660"/>
-    <property name="cos_angle_225" value="−0.7071"/>
+    <property name="cos_angle_225" value="-0.7071"/>
     <property name="cos_angle_240" value="-0.5000"/>
     <property name="cos_angle_300" value="0.5000"/>
     <property name="cos_angle_315" value="0.7071"/>
     <property name="cos_angle_330" value="0.8660"/>
+    <property name="cos_angle_345" value="0.9659"/>
     <property name="sin_angle_0" value="0.0000"/>
+    <property name="sin_angle_15" value="0.2588"/>
     <property name="sin_angle_30" value="0.5000"/>
     <property name="sin_angle_45" value="0.7071"/>
@@ -46,11 +55,14 @@
     <property name="sin_angle_135" value="0.7071"/>
     <property name="sin_angle_150" value="0.5000"/>
+    <property name="sin_angle_165" value="0.2588"/>
     <property name="sin_angle_180" value="0.0000"/>
+    <property name="sin_angle_195" value="-0.2588"/>
     <property name="sin_angle_210" value="-0.5000"/>
-    <property name="sin_angle_225" value="−0.7071"/>
+    <property name="sin_angle_225" value="-0.7071"/>
     <property name="sin_angle_240" value="-0.8660"/>
     <property name="sin_angle_300" value="-0.8660"/>
     <property name="sin_angle_315" value="-0.7071"/>
     <property name="sin_angle_330" value="-0.5000"/>
+    <property name="sin_angle_345" value="-0.2588"/>
     <!-- Component parameters -->
     <property name="ultrasonic_length" value="0.0174"/>
@@ -65,4 +77,5 @@
     <property name="battery_box_size_y" value="0.36195" />
     <property name="battery_box_size_z" value="0.0762" />
+    <property name="standoff_height" value="0.127"/>
     <!-- Note: wheel length is the wheel width -->
     <property name="wheel_length" value="0.0254" />
@@ -81,9 +94,12 @@
     <property name="baselevel_offset_y" value="0" />
     <property name="baselevel_offset_z" value="${base_size_z/2 + platter_height/2}" />
+    <!-- Note: baselevel_top_offset_z is relative to the parent -->
     <property name="baselevel_top_offset_z" value="${platter_height/2}"/>
     <!-- Middle level offset values -->
     <property name="midlevel_offset_x" value="0"/>
     <property name="midlevel_offset_y" value="0"/>
-    <property name="midlevel_offset_z" value="0"/>
+    <property name="midlevel_offset_z" value="${standoff_height + platter_height/2}"/>
+    <!-- Note: midlevel_top_offset_z is relative to the parent -->
+    <property name="midlevel_top_offset_z" value="${platter_height/2}"/>
     <!-- Top level offset values -->
     <property name="toplevel_offset_x" value="0"/>

File: src/arlobot/arlobot_description/urdf/arlobot.main.urdf.xacro (robot description, xacro)
@@ -6,5 +6,6 @@
     <xacro:include filename="$(find arlobot_description)/urdf/arlobot.base.urdf.xacro" />
     <xacro:include filename="$(find arlobot_description)/urdf/arlobot.baselevel.urdf.xacro" />
-    <!-- xacro:include filename="$(find arlobot_description)/urdf/arlobot.midlevel.urdf.xacro" />
+    <xacro:include filename="$(find arlobot_description)/urdf/arlobot.midlevel.urdf.xacro" />
+    <!--
         The midlevel includes:
             - Four supports (arlobot.support.urdf.xacro)
@@ -30,5 +31,5 @@
     <base name="base" color="Black"/>
     <baselevel parent="base" name="baselevel" color="Black"/>
-    <!-- midlevel name="midlevel" color="Black/> -->
-    <!-- toplevel name="toplevel" color="Black/> -->
+    <midlevel parent="baselevel" name="midlevel" color="Black"/>
+    <!-- <toplevel parent="base" name="toplevel" color="Black"/> -->
 </robot>
