Commit message: work on xv11 laser model

File: src/arlobot/arlobot_description/urdf/arlobot.toplevel.urdf.xacro (robot description, xacro)
@@ -61,7 +61,5 @@
     <property name="laser_offset_x" value=""/>
     <property name="laser_offset_y" value=""/>
-    <property name="laser_offset_z" value="${toplevel_top_offset_z + laser_size_z"/>
-    <laser parent="toplevel" color="DarkGrey">
-        <origin xyx="${laser_offset_x} ${laser_offset_y} ${laser_offset_z}" rpy="0 0 0 " />
-    </laser>
+    <property name="laser_offset_z" value="${toplevel_top_offset_z + laser_size_z/2"/>
+    <laser parent="toplevel" color="DarkGrey" offset_z="${laser_offset_z}"/>
 </robot>

File: src/arlobot/arlobot_description/urdf/xv11.laser.urdf.xacro (robot description, xacro)
@@ -1,35 +1,42 @@
 <?xml version="1.0"?>
-<robot name="laser" xmlns:xacro="http://ros.org/wiki/xacro">
-  <!-- A box-and-cylinder model of the Hokuyo URG-04LX-UG01 laser scanner -->
+<robot name="xv11_laser" xmlns:xacro="http://ros.org/wiki/xacro">
+  <!-- A box-and-cylinder XV11 laser scanner -->
+  <property name="xv11_laser_bottom_size_x" value="0.1238"/>
+  <property name="xv11_laser_bottom_size_y" value="0.1048"/>
+  <property name="xv11_laser_bottom_size_z" value="0.0841"/>
+  <property name="xv11_laser_disk_radius" value="0.0381"/>
+  <property name="xv11_laser_disk_height" value="0.0144"/>
+  <property name="xv11_laser_size_x" value="${xv11_laser_bottom_size_x}"/>
+  <property name="xv11_laser_size_y" value="${xv11_laser_bottom_size_y}"/>
+  <property name="xv11_laser_size_z" value="${xv11_laser_bottom_size_z + xv11_laser_disk_height}"/>
   <!-- Define the laser macro -->
-  <macro name="laser" params="parent color *origin">
+  <macro name="xv11_laser" params="parent color">
     <joint name="${parent}_laser_bottom_joint" type="fixed">
-      <xacro:insert_block name="origin" />
+      <origin xyz="0 0 0" rpy="0 0 0"/>
       <parent link="${parent}_link"/>
       <child link="base_laser_bottom"/>
     </joint>
-   <link name="base_laser_bottom">
-	 <visual>
+    <link name="base_laser_bottom">
+	  <visual>
         <origin xyz="0 0 0" rpy="0 0 0" />
         <geometry>
-          <box size="0.05 0.05 0.041" />
+          <box size="${xv11_laser_bottom_size_x} ${xv11_laser_bottom_size_y} ${xv11_laser_bottom_size_x}" />
         </geometry>
        <material name="${color}" />
-     </visual>
-     <collision>
+      </visual>
+      <collision>
         <origin xyz="0 0 0" rpy="0 0 0" />
-      <geometry>
-        <box size="0.05 0.05 0.041" />
-      </geometry>
-       </collision>
-	 <inertial>
-       <mass value="0.1" />
-         <inertia ixx="0.001" ixy="0.0" ixz="0.0"
-                   iyy="0.001" iyz="0.0"
-                   izz="0.001" />
+        <geometry>
+          <box size="${xv11_laser_bottom_size_x} ${xv11_laser_bottom_size_y} ${xv11_laser_bottom_size_x}" />
+        </geometry>
+      </collision>
+	  <inertial>
+        <mass value="0.1" />
+        <inertia ixx="0.001" ixy="0.0" ixz="0.0" iyy="0.001" iyz="0.0" izz="0.001" />
       </inertial>
-   </link>
-   <link name="base_laser_middle">
-	 <visual>
+    </link>
+    <!--
+    <link name="base_laser_middle">
+	  <visual>
         <origin xyz="0 0 0" rpy="0 0 0" />
 		<geometry>
@@ -39,17 +46,15 @@
            <color rgba="0.2 0.2 0.2 1.0"/>
         </material>
-     </visual>
-     <collision>
+      </visual>
+      <collision>
         <origin xyz="0 0 0" rpy="0 0 0" />
 		 <geometry>
           <cylinder length="0.0115" radius=".02"/>
          </geometry>
-       </collision>
-	 <inertial>
-       <mass value="0.1" />
-         <inertia ixx="0.001" ixy="0.0" ixz="0.0"
-                   iyy="0.001" iyz="0.0"
-                   izz="0.001" />
-      </inertial>
+      </collision>
+	  <inertial>
+        <mass value="0.1" />
+        <inertia ixx="0.001" ixy="0.0" ixz="0.0" iyy="0.001" iyz="0.0" izz="0.001" />
+       </inertial>
    </link>
    <joint name="base_laser_middle_joint" type="fixed">
@@ -58,4 +63,5 @@
      <origin xyz="0 0 0.02625" rpy="0 0 0" />
    </joint>
+    -->
    <link name="base_laser">
 	 <visual>
@@ -71,20 +77,18 @@
         <origin xyz="0 0 0" rpy="0 0 0" />
 		 <geometry>
-          <cylinder length="0.0175" radius=".0185"/>
+          <cylinder length="${xv11_laser_disk_height}" radius="${xv11_laser_disk_radius}"/>
          </geometry>
        </collision>
 	 <inertial>
        <mass value="0.1" />
-         <inertia ixx="0.001" ixy="0.0" ixz="0.0"
-                   iyy="0.001" iyz="0.0"
-                   izz="0.001" />
+         <inertia ixx="0.001" ixy="0.0" ixz="0.0" iyy="0.001" iyz="0.0" izz="0.001" />
       </inertial>
    </link>
    <joint name="base_laser_joint" type="fixed">
-     <parent link="base_laser_middle"/>
+     <!--<parent link="base_laser_middle"/>-->
+     <parent link="base_laser_bottom"/>
      <child link="base_laser" />
      <origin xyz="0 0 0.0145" rpy="0 0 0" />
    </joint>
   </macro>
-  <property name="laser_size_z" value="0.041 + 0.0115 + 0.0175"/>
  </robot>

Commit message: laser model

File: src/arlobot/arlobot_description/urdf/arlobot.toplevel.urdf.xacro (robot description, xacro)
@@ -62,6 +62,4 @@
     <property name="laser_offset_y" value=""/>
     <property name="laser_offset_z" value="${toplevel_top_offset_z + laser_size_z/2"/>
-    <!--
-    <laser parent="toplevel" color="DarkGrey" offset_z="${laser_offset_z}"/>
-    -->
+    <xv11_laser parent="toplevel" color="DarkGrey" offset_z="${laser_offset_z}"/>
 </robot>

File: src/arlobot/arlobot_description/urdf/xv11.laser.urdf.xacro (robot description, xacro)
@@ -18,5 +18,5 @@
     </joint>
     <link name="base_laser_bottom">
-	  <visual>
+      <visual>
         <origin xyz="0 0 0" rpy="0 0 0" />
         <geometry>
@@ -31,10 +31,9 @@
         </geometry>
       </collision>
-	  <inertial>
+      <inertial>
         <mass value="0.1" />
         <inertia ixx="0.001" ixy="0.0" ixz="0.0" iyy="0.001" iyz="0.0" izz="0.001" />
       </inertial>
     </link>
-    <!--
     <link name="base_laser_middle">
 	  <visual>
@@ -63,5 +62,4 @@
      <origin xyz="0 0 0.02625" rpy="0 0 0" />
    </joint>
-    -->
    <link name="base_laser">
 	 <visual>
@@ -86,6 +84,5 @@
    </link>
    <joint name="base_laser_joint" type="fixed">
-     <!--<parent link="base_laser_middle"/>-->
-     <parent link="base_laser_bottom"/>
+     <parent link="base_laser_middle"/>
      <child link="base_laser" />
      <origin xyz="0 0 0.0145" rpy="0 0 0" />
