Commit message: resolved modeling issues and introduced sensor array macro

File: src/arlobot/arlobot_description/urdf/arlobot.base.urdf.xacro (robot description, xacro)
@@ -1,32 +1,18 @@
 <?xml version="1.0"?>
 <robot name="base" xmlns:xacro="http://ros.org/wiki/xacro">
-    <!-- This file contains the definition for the Alrobot base which includes:
-          - the battery box (the base in this case)
-          - left/right wheels
-       Add references to the Arlobot robot system and the design files
-    -->
-    <!-- define a wheel -->
-    <macro name="wheel" params="suffix parent reflect color">
-        <joint name="${parent}_${suffix}_wheel_joint" type="continuous">
-            <axis xyz="0 0 1" />
-            <limit effort="100" velocity="100"/>
-            <safety_controller k_velocity="10" />
-            <origin xyz="${wheel_offset_x} ${reflect*wheel_offset_y} ${wheel_offset_z}" rpy="${reflect*PI/2} 0 0" />
-            <parent link="${parent}_link"/>
-            <child link="${parent}_${suffix}_wheel_link"/>
-        </joint>
-        <link name="${parent}_${suffix}_wheel_link">
+    <!-- base_footprint is a fictitious link(frame) that is on the ground
+         right below base_link origin, navigation stack depends on this frame -->
+    <!-- The base xacro macro -->
+    <macro name="base" params="color">
+        <link name="base_footprint">
             <visual>
-                <origin xyz="0 0 0" rpy="0 0 0" />
-                <geometry>
-                    <cylinder radius="${wheel_radius}" length="${wheel_length}"/>
-                </geometry>
-                <material name="${color}" />
+              <origin xyz="0 0 0" rpy="0 0 0" />
+              <geometry>
+                  <box size="0.05 0.05 0.001" />
+              </geometry>
+              <material name="TransparentGreen" />
             </visual>
         </link>
-    </macro>
-    <!-- The base xacro macro -->
-    <macro name="base" params="name color">
-        <link name="${name}_link">
+        <link name="base_link">
             <visual>
                 <origin xyz="0 0 0" rpy="0 0 0" />
@@ -43,24 +29,34 @@
             </collision>
         </link>
+        <joint name="base_joint" type="fixed">
+            <!-- Note: The wheels extend radius - z offset below the battery box so we must offset the base_joint by that same
+            amount in order for the robot to reset at 0 offset on the Z axis
+            -->
+            <origin xyz="0 0 ${base_offset_z}" rpy="0 0 0" />
+            <parent link="base_footprint"/>
+            <child link="base_link" />
+        </joint>
     </macro>
-    <link name="base_footprint">
-        <visual>
-          <origin xyz="0 0 0" rpy="0 0 0" />
-          <geometry>
-              <box size="0.05 0.05 0.001" />
-          </geometry>
-          <material name="TransparentGreen" />
-        </visual>
-    </link>
-    <joint name="base_joint" type="fixed">
-        <!-- Note: The wheels extend radius - z offset below the battery box so we must offset the base_joint by that same
-        amount in order for the robot to reset at 0 offset on the Z axis
-        -->
-        <origin xyz="0 0 ${base_offset_z}" rpy="0 0 0" />
-        <parent link="base_footprint"/>
-        <child link="base_link" />
-    </joint>
-    <!-- Add the drive wheels -->
-    <wheel parent="base" suffix="l" reflect="1" color="Orange"/>
-    <wheel parent="base" suffix="r" reflect="-1" color="Orange"/>
+    <macro name="wheel" params="parent suffix reflect color">
+        <!-- Note: type is fixed here.  tried continuous but then the link is lost.  not sure why though -->
+        <joint name="${parent}_${suffix}_wheel_joint" type="fixed">
+            <axis xyz="0 0 1" />
+            <limit effort="100" velocity="100"/>
+            <safety_controller k_velocity="10" />
+            <origin xyz="${wheel_offset_x} ${reflect*wheel_offset_y} ${wheel_offset_z}" rpy="${reflect*PI/2} 0 0" />
+            <parent link="${parent}_link"/>
+            <child link="${suffix}_wheel_link"/>
+        </joint>
+        <link name="${suffix}_wheel_link">
+            <visual>
+                <origin xyz="0 0 0" rpy="0 0 0" />
+                <geometry>
+                    <cylinder radius="${wheel_radius}" length="${wheel_length}"/>
+                </geometry>
+                <material name="${color}" />
+            </visual>
+        </link>
+    </macro>
+    <wheel parent="base" suffix="left" reflect="1" color="Orange"/>
+    <wheel parent="base" suffix="right" reflect="-1" color="Orange"/>
 </robot>

File: src/arlobot/arlobot_description/urdf/arlobot.baselevel.urdf.xacro (robot description, xacro)
@@ -199,4 +199,47 @@
         </link>
     </macro>
+    <!-- Note: The following macros are purely organizational in nature.  That is, they do not contribute to the
+               geometry of the model.  They only wrap the sensor macros so they are grouped by function and position
+    -->
+    <macro name="baselevel_front_ultrasonic_array" params="offset_z">
+        <link name="baselevel_front_ultrasonic_array_link">
+            <!-- This is an organizational link it has no dimensions -->
+        </link>
+        <joint name="baselevel_front_ultrasonic_array_joint" type="fixed">
+            <parent link="baselevel_link"/>
+            <child link="baselevel_front_ultrasonic_array_link"/>
+        </joint>
+        <ultrasonic_array_5_front parent="baselevel_front_ultrasonic_array" offset_z="${offset_z}"/>
+    </macro>
+    <macro name="baselevel_back_ultrasonic_array" params="offset_z">
+        <link name="baselevel_back_ultrasonic_array_link">
+            <!-- This is an organizational link it has no dimensions -->
+        </link>
+        <joint name="baselevel_back_ultrasonic_array_joint" type="fixed">
+            <parent link="baselevel_link"/>
+            <child link="baselevel_back_ultrasonic_array_link"/>
+        </joint>
+        <ultrasonic_array_5_back parent="baselevel_back_ultrasonic_array" offset_z="${offset_z}"/>
+    </macro>
+    <macro name="baselevel_front_infrared_array" params="offset_z">
+        <link name="baselevel_front_infrared_array_link">
+            <!-- This is an organizational link it has no dimensions -->
+        </link>
+        <joint name="baselevel_front_infrared_array_joint" type="fixed">
+            <parent link="baselevel_link"/>
+            <child link="baselevel_front_infrared_array_link"/>
+        </joint>
+        <infrared_array_2_front_lower parent="baselevel_front_infrared_array" offset_z="${offset_z}"/>
+    </macro>
+    <macro name="baselevel_back_infrared_array" params="offset_z">
+        <link name="baselevel_back_infrared_array_link">
+            <!-- This is an organizational link it has no dimensions -->
+        </link>
+        <joint name="baselevel_back_infrared_array_joint" type="fixed">
+            <parent link="baselevel_link"/>
+            <child link="baselevel_back_infrared_array_link"/>
+        </joint>
+        <infrared_array_2_back_lower parent="baselevel_back_infrared_array" offset_z="${offset_z}"/>
+    </macro>
     <!--
     Build the Base Level
@@ -207,10 +250,10 @@
     <!-- This calculation is needed to position the ultrasonic sensor on the top of the base level platter -->
     <property name="baselevel_ultrasonic_offset_z" value="${baselevel_top_offset_z + ultrasonic_height/2}"/>
-    <ultrasonic_array_5_front parent="baselevel" offset_z="${baselevel_ultrasonic_offset_z}"/>
-    <ultrasonic_array_5_back parent="baselevel" offset_z="${baselevel_ultrasonic_offset_z}"/>
+    <baselevel_front_ultrasonic_array offset_z="${baselevel_ultrasonic_offset_z}"/>
+    <baselevel_back_ultrasonic_array offset_z="${baselevel_ultrasonic_offset_z}"/>
     <!-- This calculation is needed to position the infrared sensor under the base level platter -->
     <property name="baselevel_infrared_offset_z" value="${-platter_height - infrared_height/2}"/>
-    <infrared_array_2_front_lower parent="baselevel" offset_z="${baselevel_infrared_offset_z}"/>
-    <infrared_array_2_back_lower parent="baselevel" offset_z="${baselevel_infrared_offset_z}"/>
+    <baselevel_front_infrared_array offset_z="${baselevel_infrared_offset_z}"/>
+    <baselevel_back_infrared_array offset_z="${baselevel_infrared_offset_z}"/>
     <power parent="baselevel" color="LightGrey"/>
     <motor_driver parent="baselevel" suffix="left" color="Orange" offset_x="${left_motor_driver_offset_x}" offset_y="${left_motor_driver_offset_y}" offset_z="${left_motor_driver_offset_z}"  yaw="${angle_315}"/>

File: src/arlobot/arlobot_description/urdf/arlobot.main.urdf.xacro (robot description, xacro)
@@ -4,10 +4,13 @@
     <xacro:include filename="$(find arlobot_description)/urdf/materials.urdf.xacro" />
     <xacro:include filename="$(find arlobot_description)/urdf/arlobot.global.urdf.xacro"/>
+    <!--
     <xacro:include filename="$(find arlobot_description)/urdf/arlobot.base.urdf.xacro" />
+    -->
+    <xacro:include filename="$(find arlobot_description)/urdf/arlobot.newbase.urdf.xacro" />
     <xacro:include filename="$(find arlobot_description)/urdf/arlobot.baselevel.urdf.xacro" />
     <xacro:include filename="$(find arlobot_description)/urdf/arlobot.midlevel.urdf.xacro" />
     <xacro:include filename="$(find arlobot_description)/urdf/arlobot.toplevel.urdf.xacro" />
-    <!-- Add the base and wheels -->
-    <base name="base" color="Black"/>
+    <!-- Add each level of the robot -->
+    <base color="Black"/>
     <baselevel parent="base" name="baselevel" color="Black"/>
     <midlevel parent="baselevel" name="midlevel" color="Black"/>

File: src/arlobot/arlobot_description/urdf/arlobot.midlevel.urdf.xacro (robot description, xacro)
@@ -67,4 +67,47 @@
         </link>
     </macro>
+    <!-- Note: The following macros are purely organizational in nature.  That is, they do not contribute to the
+               geometry of the model.  They only wrap the sensor macros so they are grouped by function and position
+    -->
+    <macro name="midlevel_front_ultrasonic_array" params="offset_z">
+        <link name="midlevel_front_ultrasonic_array_link">
+            <!-- This is an organizational link it has no dimensions -->
+        </link>
+        <joint name="midlevel_front_ultrasonic_array_joint" type="fixed">
+            <parent link="midlevel_link"/>
+            <child link="midlevel_front_ultrasonic_array_link"/>
+        </joint>
+        <ultrasonic_array_3_front parent="midlevel_front_ultrasonic_array" offset_z="${offset_z}"/>
+    </macro>
+    <macro name="midlevel_back_ultrasonic_array" params="offset_z">
+        <link name="midlevel_back_ultrasonic_array_link">
+            <!-- This is an organizational link it has no dimensions -->
+        </link>
+        <joint name="midlevel_back_ultrasonic_array_joint" type="fixed">
+            <parent link="midlevel_link"/>
+            <child link="midlevel_back_ultrasonic_array_link"/>
+        </joint>
+        <ultrasonic_array_3_back parent="midlevel_back_ultrasonic_array" offset_z="${offset_z}"/>
+    </macro>
+    <macro name="midlevel_front_infrared_array" params="offset_z">
+        <link name="midlevel_front_infrared_array_link">
+            <!-- This is an organizational link it has no dimensions -->
+        </link>
+        <joint name="midlevel_front_infrared_array_joint" type="fixed">
+            <parent link="midlevel_link"/>
+            <child link="midlevel_front_infrared_array_link"/>
+        </joint>
+        <infrared_array_4_front parent="midlevel_front_infrared_array" offset_z="${offset_z}"/>
+    </macro>
+    <macro name="midlevel_back_infrared_array" params="offset_z">
+        <link name="midlevel_back_infrared_array_link">
+            <!-- This is an organizational link it has no dimensions -->
+        </link>
+        <joint name="midlevel_back_infrared_array_joint" type="fixed">
+            <parent link="midlevel_link"/>
+            <child link="midlevel_back_infrared_array_link"/>
+        </joint>
+        <infrared_array_4_back parent="midlevel_back_infrared_array" offset_z="${offset_z}"/>
+    </macro>
     <!--
     Build the Mid Level
@@ -83,10 +126,10 @@
     <!-- This calculation is needed to position the ultrasonic sensor on the top of the mid level platter -->
     <property name="midlevel_ultrasonic_offset_z" value="${midlevel_top_offset_z + ultrasonic_height/2}"/>
-    <ultrasonic_array_3_front parent="midlevel" offset_z="${midlevel_ultrasonic_offset_z}"/>
-    <ultrasonic_array_3_back  parent="midlevel" offset_z="${midlevel_ultrasonic_offset_z}"/>
+    <midlevel_front_ultrasonic_array offset_z="${midlevel_ultrasonic_offset_z}"/>
+    <midlevel_back_ultrasonic_array offset_z="${midlevel_ultrasonic_offset_z}"/>
     <!-- This calculation is needed to position the infrared sensor under the mid level platter -->
     <property name="midlevel_infrared_offset_z" value="${-(infrared_height/2 + platter_height/2)}"/>
-    <infrared_array_4_front parent="midlevel" offset_z="${midlevel_infrared_offset_z}"/>
-    <infrared_array_4_back parent="midlevel" offset_z="${midlevel_infrared_offset_z}"/>
+    <midlevel_front_infrared_array offset_z="${midlevel_infrared_offset_z}"/>
+    <midlevel_back_infrared_array offset_z="${midlevel_infrared_offset_z}"/>
     <pc_case parent="midlevel" color="Blue"/>
 </robot>

File: src/arlobot/arlobot_description/urdf/arlobot.toplevel.urdf.xacro (robot description, xacro)
@@ -41,4 +41,27 @@
         </link>
     </macro>
+    <!-- Note: The following macros are purely organizational in nature.  That is, they do not contribute to the
+               geometry of the model.  They only wrap the sensor macros so they are grouped by function and position
+    -->
+    <macro name="toplevel_front_infrared_array" params="offset_z">
+        <link name="toplevel_front_infrared_array_link">
+            <!-- This is an organizational link it has no dimensions -->
+        </link>
+        <joint name="toplevel_front_infrared_array_joint" type="fixed">
+            <parent link="toplevel_link"/>
+            <child link="toplevel_front_infrared_array_link"/>
+        </joint>
+        <infrared_array_2_front_upper parent="toplevel_front_infrared_array" offset_z="${offset_z}"/>
+    </macro>
+    <macro name="toplevel_back_infrared_array" params="offset_z">
+        <link name="toplevel_back_infrared_array_link">
+            <!-- This is an organizational link it has no dimensions -->
+        </link>
+        <joint name="toplevel_back_infrared_array_joint" type="fixed">
+            <parent link="toplevel_link"/>
+            <child link="toplevel_back_infrared_array_link"/>
+        </joint>
+        <infrared_array_2_back_upper parent="toplevel_back_infrared_array" offset_z="${offset_z}"/>
+    </macro>
     <!--
     Build the Top Level
@@ -57,6 +80,6 @@
     <!-- This calculation is needed to position the infrared sensor under the top level platter -->
     <property name="toplevel_infrared_offset_z" value="${-(infrared_height/2 + platter_height/2)}"/>
-    <infrared_array_2_front_upper parent="toplevel" offset_z="${toplevel_infrared_offset_z}"/>
-    <infrared_array_2_back_upper parent="toplevel" offset_z="${toplevel_infrared_offset_z}"/>
+    <toplevel_front_infrared_array offset_z="${toplevel_infrared_offset_z}"/>
+    <toplevel_back_infrared_array offset_z="${toplevel_infrared_offset_z}"/>
     <property name="laser_offset_x" value=""/>
     <property name="laser_offset_y" value=""/>
